File: pcb/pcb.kicad_pcb (KiCad board)
At the start: 2 copper layers, 1 part

Commit message: done final pcb
Parts:
- removed REF**: RP2350A-ZERO, Custom_modules:RP2350A-ZERO
- added J1: Conn_Coaxial, Custom_modules:BNC-connector, F.Cu at (138.7, 126.4)
- added J2: RP2350A-ZERO, Custom_modules:RP2350A-ZERO, F.Cu at (159.0, 90.2)
- added K1: G6K-2F-Y DC3, Relay_SMD:Relay_DPDT_Omron_G6K-2F-Y, F.Cu at (135.0, 108.7)
- added K2: G6K-2F-Y DC3, Relay_SMD:Relay_DPDT_Omron_G6K-2F-Y, F.Cu at (159.0, 108.7)
- added R10: 10k, Resistor_SMD:R_0603_1608Metric_Pad0.98x0.95mm_HandSolder, F.Cu at (169.1, 112.0)
- added R11: 10k, Resistor_SMD:R_0603_1608Metric_Pad0.98x0.95mm_HandSolder, F.Cu at (164.5, 121.5)
- added R12: 10k, Resistor_SMD:R_0603_1608Metric_Pad0.98x0.95mm_HandSolder, F.Cu at (164.5, 126.5)
- added R7: 1.62M, Resistor_SMD:R_2010_5025Metric_Pad1.40x2.65mm_HandSolder, F.Cu at (147.0, 105.0)
- added R8: 16.2k, Resistor_SMD:R_0603_1608Metric_Pad0.98x0.95mm_HandSolder, F.Cu at (169.0, 105.5)
- added R9: 100k, Resistor_SMD:R_0805_2012Metric_Pad1.20x1.40mm_HandSolder, F.Cu at (145.5, 112.0)
- added U1: ADC121S021CIMF, Package_TO_SOT_SMD:SOT-23-6_Handsoldering, F.Cu at (135.5, 84.9)
- added U2: PGA113, Package_SO:TSSOP-10_3x3mm_P0.5mm, F.Cu at (135.5, 95.4)
- added U6: LM321, Package_TO_SOT_SMD:SOT-23-5_HandSoldering, F.Cu at (156.2, 122.5)
Routing:
- net GND: track 0.00 -> 156.9 mm, vias 0 -> 6
- net +3V3: track 0.00 -> 106.2 mm, vias 0 -> 5
- net /1V65: track 0.00 -> 68.7 mm, vias 0 -> 5
- net Net-(U2-CH0/V_{CAL}): track 0.00 -> 54.7 mm
- net Net-(J1-In): track 0.00 -> 41.5 mm, vias 0 -> 1
- net /adc_sda: track 0.00 -> 34.4 mm
- net /pga_slck: track 0.00 -> 33.6 mm, vias 0 -> 2
- net /adc_scl: track 0.00 -> 32.3 mm
- net /pga_dio: track 0.00 -> 32.0 mm, vias 0 -> 2
- net /pga_cs: track 0.00 -> 30.9 mm, vias 0 -> 2
- net Net-(K1-Pad4): track 0.00 -> 24.3 mm
- net Net-(J2-Pin_8): track 0.00 -> 20.9 mm, vias 0 -> 2
- net /50V_relay: track 0.00 -> 20.4 mm
- net Net-(K2-Pad2): track 0.00 -> 16.1 mm
- net /5V_relay: track 0.00 -> 15.6 mm
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Other:
- board outline added: 44.5 x 58 mm
