File: pcb/pcb.kicad_sch (KiCad schematic)
At the start: 0 parts

Commit message: added pcb files
Parts:
- added J1: Conn_Coaxial, symbol Connector:Conn_Coaxial
- added K1: G6K-2, symbol Relay:G6K-2
- added U1: RP2350A, Package_DFN_QFN:QFN-60-1EP_7x7mm_P0.4mm_EP3.4x3.4mm, symbol MCU_RaspberryPi:RP2350A
- added U2: PGA113, Package_SO:TSSOP-10_3x3mm_P0.5mm, symbol Analog:PGA113
- added U3: ADC121C021CIMM, Package_SO:MSOP-8_3x3mm_P0.65mm, symbol Analog_ADC:ADC121C021CIMM
Connections:
- new net: U1.1 (IOVDD), U1.11 (IOVDD), U1.20 (IOVDD), U1.30 (IOVDD), U1.38 (IOVDD), U1.45 (IOVDD)
- new net: U1.23 (DVDD), U1.39 (DVDD), U1.6 (DVDD)

Commit message: updated pcb  schematic
Parts:
- added C1, C2: 15pF, symbol Device:C
- added C3, C4: 10u, symbol Device:C
- added C5, C7: 4.7u, Package_QFP:TQFP-44_10x10mm_P0.8mm, symbol Device:C
- added C6: 4.7u, symbol Device:C
- added J2: USB_C_Receptacle_USB2.0_14P, Package_TO_SOT_SMD:SOT-223-3_TabPin2, symbol Connector:USB_C_Receptacle_USB2.0_14P
- added J3: Conn_02x05_Odd_Even, symbol Connector_Generic:Conn_02x05_Odd_Even
- added K2: G6K-2, symbol Relay:G6K-2
- added L1: 3.3u, symbol Device:L
- added R1: 1k, symbol Device:R
- added R2, R3: 27, symbol Device:R
- added R4, R5: 5.1k, symbol Device:R
- added R6: 33, symbol Device:R
- added SW1, SW2: SW_Push, Button_Switch_THT:SW_NKK_GW12LJP, symbol Switch:SW_Push
- added TP1: TestPoint, symbol Connector:TestPoint
- added U4: W25Q128JVE, Package_SON:WSON-8-1EP_8x6mm_P1.27mm_EP3.4x4.3mm, symbol Memory_Flash:W25Q128JVE
- added U5: NCP1117-3.3_SOT223, Package_TO_SOT_SMD:SOT-223-3_TabPin2, symbol Regulator_Linear:NCP1117-3.3_SOT223
- added Y1: 12MHz, Package_SON:WSON-8-1EP_8x6mm_P1.27mm_EP3.4x4.3mm, symbol Device:Crystal
Connections:
- net at U1.1 (IOVDD), U1.11 (IOVDD), U1.20 (IOVDD)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: now also U1.44 (ADC_AVDD), U1.49 (VREG_VIN), U1.53 (USB_OTP_VDD), U1.54 (QSPI_IOVDD), C4.1, C7.1, R6.1, U5.2 (VO)
- net at U1.21 (XIN): now also C1.2, Y1.2
- net at U1.22 (XOUT): now also C2.1, R1.1, R1.2, Y1.1
- net at U1.23 (DVDD), U1.39 (DVDD), U1.6 (DVDD): now also U1.50 (VREG_FB), C6.2, L1.2
- net at U1.46 (VREG_AVDD): now also C5.2, R6.2
- net at U1.48 (VREG_LX): now also L1.1
- net at U1.51 (USB_DM): now also R2.2
- net at U1.52 (USB_DP): now also R3.2
- new net: J2.B5 (CC2), R5.1
- new net: J2.A5 (CC1), R4.1
- new net: J2.A6 (D+), J2.B6 (D+), R3.1
- new net: J2.A7 (D-), J2.B7 (D-), R2.1
- new net +5V: C3.1, J2.A4 (VBUS), J2.A9 (VBUS), J2.B4 (VBUS), J2.B9 (VBUS), U5.3 (VI)
- new net GND: C1.1, C2.2, C3.2, C4.2, C5.1, C6.1, C7.2, J2.A1 (GND), J2.A12 (GND), J2.B1 (GND), J2.B12 (GND), J2.SH (SHIELD), R4.2, R5.2, U5.1 (GND)
- no-connect marks 0 -> 1
Other:
- company: (none) -> MITBLR
- title: (none) -> Oscilloscope
- moved on the sheet: J1, K1, U1, U2, U3

Commit message: afe design
Parts:
- added R10: 16.2k, symbol Device:R
- added R11, R12, R8: 10k, symbol Device:R
- added R7: 100k, symbol Device:R
- added R9: 1.62M, symbol Device:R
- added U6: LM321, Package_TO_SOT_SMD:SOT-23-5, symbol Amplifier_Operational:LM321
Connections:
- net GND: now also J1.2 (Ext), U2.6 (GND), U3.7 (GND), R11.2, U6.2 (V-)
- net at C4.1, C7.1, R6.1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: now also U2.1 (AV_{DD}), U2.10 (DV_{DD}), R12.1, U6.5 (V+)
- net at U2.3 (CH0/V_{CAL}): now also K1.5, K2.7
- net at U2.4 (V_{REF}): now also R10.1, R9.1, U6.3 (-), U6.4
- net at U2.5 (V_{OUT}): now also U3.4 (VIN)
- net at J1.1 (In): now also K1.3, K2.3
- net at K2.2: now also R8.2
- net at K2.6: now also R10.2, R8.1
- net at K1.4: now also R7.2
- net at K1.6: now also R7.1, R9.2
- new net: R11.1, R12.2, U6.1 (+)
Other:
- note added: "50vpp"
- note added: "5vpp"
- moved on the sheet: C1, C2, C3, C4, C5, C6, C7, J1, J2, J3, K1, K2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

Commit message: updated pcb
Parts:
- removed C1, C2: 15pF, symbol Device:C
- removed C3, C4: 10u, symbol Device:C
- removed C5, C7: 4.7u, Package_QFP:TQFP-44_10x10mm_P0.8mm, symbol Device:C
- removed C6: 4.7u, symbol Device:C
- removed J2: USB_C_Receptacle_USB2.0_14P, Package_TO_SOT_SMD:SOT-223-3_TabPin2, symbol Connector:USB_C_Receptacle_USB2.0_14P
- removed J3: Conn_02x05_Odd_Even, symbol Connector_Generic:Conn_02x05_Odd_Even
- removed L1: 3.3u, symbol Device:L
- removed R1: 1k, symbol Device:R
- removed R2, R3: 27, symbol Device:R
- removed R4, R5: 5.1k, symbol Device:R
- removed R6: 33, symbol Device:R
- removed SW1, SW2: SW_Push, Button_Switch_THT:SW_NKK_GW12LJP, symbol Switch:SW_Push
- removed TP1: TestPoint, symbol Connector:TestPoint
- removed U1: RP2350A, Package_DFN_QFN:QFN-60-1EP_7x7mm_P0.4mm_EP3.4x3.4mm, symbol MCU_RaspberryPi:RP2350A
- removed U4: W25Q128JVE, Package_SON:WSON-8-1EP_8x6mm_P1.27mm_EP3.4x4.3mm, symbol Memory_Flash:W25Q128JVE
- removed U5: NCP1117-3.3_SOT223, Package_TO_SOT_SMD:SOT-223-3_TabPin2, symbol Regulator_Linear:NCP1117-3.3_SOT223
- removed Y1: 12MHz, Package_SON:WSON-8-1EP_8x6mm_P1.27mm_EP3.4x4.3mm, symbol Device:Crystal
- added J2: RP2350A-ZERO, Custom_modules:RP2350A-ZERO, symbol Connector_Generic:Conn_01x23
- added U7: NCP1117-3.3_SOT223, Package_TO_SOT_SMD:SOT-223-3_TabPin2, symbol Regulator_Linear:NCP1117-3.3_SOT223
- K1, K2: value G6K-2 -> G6K-2F-Y DC3; footprint (none) -> Relay_SMD:Relay_DPDT_Omron_G6K-2F-Y
Connections:
- net +3V3: now reaches R12.1, U2.1 (AV_{DD}), U2.10 (DV_{DD}), U6.5 (V+)
- net +3V3: now also U3.5 (VA)
- net pga_slck: now reaches U2.7 (SCLK)
- net pga_slck: now also J2.3 (Pin_3)
- net pga_dio: now reaches U2.8 (DIO)
- net pga_dio: now also J2.4 (Pin_4)
- net pga_cs: now reaches U2.9 (~{CS})
- net pga_cs: now also J2.5 (Pin_5)
- net adc_scl: now reaches U3.1 (SCL)
- net adc_scl: now also J2.2 (Pin_2)
- net at U3.2 (ALERT): now also J2.8 (Pin_8)
- net adc_sda: now reaches U3.8 (SDA)
- net adc_sda: now also J2.1 (Pin_1)
- no-connect marks 1 -> 0

Commit message: schematic connections done
Parts:
- R10: value 16.2k -> 10k
- R7: value 100k -> 1.62M
- R8: value 10k -> 16.2k
- R9: value 1.62M -> 100k
Connections:
- net +3V3 is gone; now on net 3V3: R12.1, U2.1 (AV_{DD}), U2.10 (DV_{DD}), U3.5 (VA), U6.5 (V+)
- net GND: now also J2.22 (Pin_22), K1.8, K2.8, U3.3 (ADR0), U3.6 (ADR1)
- net 1V65: now reaches R10.1, R9.1, U2.4 (V_{REF}), U6.3 (-), U6.4
- net 5V_relay: now reaches K2.1
- net 5V_relay: now also J2.11 (Pin_11)
- net 50V_relay: now reaches K1.1
- net 50V_relay: now also J2.12 (Pin_12)
- net 3V3: now reaches J2.21 (Pin_21)
Other:
- moved on the sheet: J2

Commit message: done final pcb
Parts:
- removed U3: ADC121C021CIMM, Package_SO:MSOP-8_3x3mm_P0.65mm, symbol Analog_ADC:ADC121C021CIMM
- removed U7: NCP1117-3.3_SOT223, Package_TO_SOT_SMD:SOT-223-3_TabPin2, symbol Regulator_Linear:NCP1117-3.3_SOT223
- added U1: ADC121S021CIMF, Package_TO_SOT_SMD:SOT-23-6_Handsoldering, symbol Analog_ADC:ADC121S021CIMF
- J1: footprint (none) -> Custom_modules:BNC-connector
- R10, R11, R12, R8: footprint (none) -> Resistor_SMD:R_0603_1608Metric_Pad0.98x0.95mm_HandSolder
- R7: footprint (none) -> Resistor_SMD:R_2010_5025Metric_Pad1.40x2.65mm_HandSolder
- R9: footprint (none) -> Resistor_SMD:R_0805_2012Metric_Pad1.20x1.40mm_HandSolder
- U6: footprint Package_TO_SOT_SMD:SOT-23-5 -> Package_TO_SOT_SMD:SOT-23-5_HandSoldering
Connections:
- net 50V_relay: now also J2.11 (Pin_12); no longer J2.12 (Pin_12)
- net 5V_relay: now also J2.10 (Pin_11); no longer J2.11 (Pin_11)
- net GND: now also J2.GND (Pin_22), U1.2 (GND); no longer J2.22 (Pin_22)
- net adc_scl: now also J2.1 (Pin_2), U1.4 (SCLK); no longer J2.2 (Pin_2)
- net adc_sda: now also J2.0 (Pin_1), U1.5 (SDO); no longer J2.1 (Pin_1)
- net pga_cs: now also J2.4 (Pin_5); no longer J2.5 (Pin_5)
- net pga_dio: now also J2.3 (Pin_4); no longer J2.4 (Pin_4)
- net pga_slck: now also J2.2 (Pin_3); no longer J2.3 (Pin_3)
- net at U2.5 (V_{OUT}): now also U1.3 (VIN)
- net at J2.7 (Pin_8): now also U1.6 (CS_N)
- net 3V3 renamed +3V3
- net +3V3: now also J2.3V3 (Pin_21), U1.1 (VDD); no longer J2.21 (Pin_21)
- no-connect marks 0 -> 18
Other:
- moved on the sheet: J2
